File: treat-dispenser.brd (EAGLE design)
At the start: 88.9 x 44.5 mm, 10 parts, among them U1 ARDUINO_PRO_MINI, U2 PB1000

Commit message: eagle and arduino update for servo with feedback sensor
Parts:
- removed JP3: (no value), SparkFun-Connectors:1X03
- added J1: (no value), SparkFun-Connectors:1X04
Connections:
- new net FB: J1.4, U1.17
- net 5V: now also J1.2; no longer JP3.2
- net GND: now also J1.1; no longer JP3.1
- net SERVO: now also J1.3; no longer JP3.3
Routing:
- net FB: track 0.00 -> 76.7 mm
Changed lines of the file:
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@@
 <attribute name="VALUE" x="86.36" y="27.94" size="0.4064" layer="27" rot="R180"/>
-</element>
-<element name="JP3" library="SparkFun-Connectors" package="1X03" value="" x="5.08" y="12.7" smashed="yes" rot="R90">
-<attribute name="PN" value="952-1312-ND" x="5.08" y="12.7" size="1.778" layer="27" rot="R90" display="off"/>
-<attribute name="NAME" x="6.2992" y="8.9408" size="1.27" layer="25" font="vector" align="bottom-right"/>
-<attribute name="VALUE" x="8.255" y="11.43" size="1.27" layer="27" rot="R90"/>
 </element>
 <element name="JP4" library="SparkFun-Connectors" package="1X02" value="" x="59.69" y="35.56" smashed="yes">
@@
 <attribute name="VALUE" x="33.02" y="32.385" size="1.27" layer="27"/>
 </element>
+<element name="J1" library="SparkFun-Connectors" package="1X04" value="" x="5.08" y="12.7" rot="R90">
+<attribute name="PROD_ID" value="CONN-09696" x="5.08" y="12.7" size="1.778" layer="27" rot="R90" display="off"/>
+</element>
 </elements>
 <signals>
 <signal name="GND" class="1">
-<contactref element="JP3" pad="1"/>
 <contactref element="JP2" pad="SLEEVE"/>
 <polygon width="0.3556" layer="16">
@@
 <contactref element="JP5" pad="1"/>
 <contactref element="JP6" pad="1"/>
+<contactref element="J1" pad="1"/>
 </signal>
 <signal name="SERVO">
-<contactref element="JP3" pad="3"/>
 <contactref element="U1" pad="9"/>
 <wire x1="62.23" y1="14.605" x2="57.785" y2="10.16" width="0.4064" layer="1"/>
 <wire x1="57.785" y1="10.16" x2="12.7" y2="10.16" width="0.4064" layer="1"/>
-<wire x1="5.08" y1="17.78" x2="12.7" y2="10.16" width="0.4064" layer="1"/>
+<contactref element="J1" pad="3"/>
+<wire x1="12.7" y1="10.16" x2="5.08" y2="17.78" width="0.4064" layer="1"/>
 </signal>
 <signal name="N$9">
@@
 </signal>
 <signal name="5V">
-<contactref element="JP3" pad="2"/>
 <contactref element="U2" pad="P8"/>
 <contactref element="U1" pad="24"/>
@@
 <wire x1="41.91" y1="29.845" x2="41.91" y2="40.64" width="0.8128" layer="16"/>
 <wire x1="30.607" y1="34.671" x2="30.607" y2="40.64" width="0.8128" layer="16"/>
-<wire x1="2.54" y1="27.305" x2="2.54" y2="40.64" width="0.8128" layer="16"/>
-<wire x1="2.54" y1="27.305" x2="2.54" y2="17.78" width="0.8128" layer="16"/>
-<wire x1="2.54" y1="17.78" x2="5.08" y2="15.24" width="0.8128" layer="16"/>
+<contactref element="J1" pad="2"/>
+<wire x1="5.08" y1="15.24" x2="2.54" y2="17.78" width="0.8128" layer="16"/>
+<wire x1="2.54" y1="17.78" x2="2.54" y2="40.64" width="0.8128" layer="16"/>
 </signal>
 <signal name="B2">
@@
 <wire x1="55.88" y1="35.56" x2="59.69" y2="35.56" width="0.4064" layer="1"/>
 </signal>
+<signal name="FB">
+<contactref element="J1" pad="4"/>
+<contactref element="U1" pad="17"/>
+<wire x1="3.81" y1="21.59" x2="3.81" y2="33.02" width="0.4064" layer="1"/>
+<wire x1="3.81" y1="33.02" x2="11.43" y2="40.64" width="0.4064" layer="1"/>
+<wire x1="11.43" y1="40.64" x2="36.83" y2="40.64" width="0.4064" layer="1"/>
+<wire x1="36.83" y1="40.64" x2="44.45" y2="33.02" width="0.4064" layer="1"/>
+<wire x1="44.45" y1="33.02" x2="56.515" y2="33.02" width="0.4064" layer="1"/>
+<wire x1="59.69" y1="29.845" x2="56.515" y2="33.02" width="0.4064" layer="1"/>
+<wire x1="5.08" y1="20.32" x2="3.81" y2="21.59" width="0.4064" layer="1"/>
+</signal>
 </signals>
