File: treat-dispenser.sch (EAGLE design)
At the start: 10 parts, among them U1 ARDUINO_PRO_MINI, U2 PB1000

Commit message: eagle and arduino update for servo with feedback sensor
Parts:
- removed JP3: (no value), SparkFun-Connectors:M03PTH
- added J1: (no value), SparkFun-Connectors:M04PTH
Connections:
- new net FB: J1.4, U1.A0
- net 5V: now also J1.2; no longer JP3.2
- net GND: now also J1.1; no longer JP3.1
- net SERVO: now also J1.3; no longer JP3.3
Changed lines of the file:
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@@
 <attribute name="PN" value="CP1-3523N-ND"/>
-</part>
-<part name="JP3" library="SparkFun-Connectors" deviceset="M03" device="PTH">
-<attribute name="PN" value="952-1312-ND"/>
 </part>
 <part name="GND10" library="supply1" deviceset="GND" device=""/>
@@
 <part name="GND6" library="supply1" deviceset="GND" device=""/>
 <part name="GND7" library="supply1" deviceset="GND" device=""/>
+<part name="J1" library="SparkFun-Connectors" deviceset="M04" device="PTH"/>
 </parts>
 <sheets>
@@
 <attribute name="PN" x="12.7" y="127" size="1.778" layer="96" rot="MR180" display="off"/>
 </instance>
-<instance part="JP3" gate="G$1" x="10.16" y="106.68">
-<attribute name="PN" x="10.16" y="106.68" size="1.778" layer="96" display="off"/>
-</instance>
 <instance part="GND10" gate="1" x="20.32" y="99.06"/>
 <instance part="GND12" gate="1" x="22.86" y="119.38"/>
@@
 <instance part="GND6" gate="1" x="60.96" y="76.2"/>
 <instance part="GND7" gate="1" x="22.86" y="134.62"/>
+<instance part="J1" gate="G$1" x="12.7" y="106.68"/>
 </instances>
 <busses>
@@
 <net name="GND" class="1">
 <segment>
-<pinref part="JP3" gate="G$1" pin="1"/>
 <pinref part="GND10" gate="1" pin="GND"/>
 <wire x1="17.78" y1="104.14" x2="20.32" y2="104.14" width="0.1524" layer="91"/>
 <wire x1="20.32" y1="104.14" x2="20.32" y2="101.6" width="0.1524" layer="91"/>
+<pinref part="J1" gate="G$1" pin="1"/>
 </segment>
 <segment>
@@
 <net name="SERVO" class="0">
 <segment>
-<pinref part="JP3" gate="G$1" pin="3"/>
 <wire x1="17.78" y1="109.22" x2="25.4" y2="109.22" width="0.1524" layer="91"/>
 <label x="17.78" y="109.22" size="1.778" layer="95"/>
+<pinref part="J1" gate="G$1" pin="3"/>
 </segment>
 <segment>
@@
 <net name="5V" class="0">
 <segment>
-<pinref part="JP3" gate="G$1" pin="2"/>
 <wire x1="17.78" y1="106.68" x2="27.94" y2="106.68" width="0.1524" layer="91"/>
 <wire x1="27.94" y1="106.68" x2="27.94" y2="111.76" width="0.1524" layer="91"/>
 <pinref part="SUPPLY1" gate="G$1" pin="5V"/>
+<pinref part="J1" gate="G$1" pin="2"/>
 </segment>
 <segment>
@@
 </segment>
 </net>
+<net name="FB" class="0">
+<segment>
+<pinref part="J1" gate="G$1" pin="4"/>
+<wire x1="17.78" y1="111.76" x2="25.4" y2="111.76" width="0.1524" layer="91"/>
+<label x="17.78" y="111.76" size="1.778" layer="95"/>
+</segment>
+<segment>
+<pinref part="U1" gate="G$1" pin="A0"/>
+<wire x1="71.12" y1="162.56" x2="78.74" y2="162.56" width="0.1524" layer="91"/>
+<label x="73.66" y="162.56" size="1.778" layer="95"/>
+</segment>
+</net>
